Commit message: fixes

File: urdf/inc/create_link.xacro (robot description, xacro)
@@ -5,5 +5,9 @@
         xyz_offset
         rpy_offset
-        mesh_name">
+        mesh_name
+        ixx
+        iyy
+        izz
+        mass">
     <link name="${link_name}">
       <visual>
@@ -20,6 +24,6 @@
       </collision>
       <inertial>
-        <mass value="1"/>
-        <inertia ixx="1.0" ixy="0.0" ixz="0.0" iyy="1.0" iyz="0.0" izz="1.0"/>
+        <mass value="${mass}"/>
+        <inertia ixx="${ixx}" ixy="0.0" ixz="0.0" iyy="${iyy}" iyz="0.0" izz="${izz}"/>
       </inertial>
     </link>

File: urdf/mercury.ros2_control.xacro (robot description, xacro)
@@ -4,5 +4,5 @@
     <ros2_control name="${name}" type="system">
       <hardware>
-        <plugin>tr_robot/RobotSystem</plugin>
+        <plugin>tr_hardware_interface/RobotSystem</plugin>
       </hardware>
       <joint name="joint_1">

File: urdf/mercury_description.urdf.xacro (robot description, xacro)
@@ -8,4 +8,8 @@
       rpy_offset="0 0 0"
       mesh_name="ROS2_Base"
+      ixx="0.00443333156"
+      iyy="0.00443333156"
+      izz="0.0072"
+      mass="4.0"
   />
   <xacro:create_link
@@ -14,4 +18,8 @@
       rpy_offset="0 0 0"
       mesh_name="ROS2_J1"
+      ixx="0.010267495893"
+      iyy="0.010267495893"
+      izz="0.00666"
+      mass="3.7"
   />
   <xacro:create_link
@@ -20,4 +28,8 @@
       rpy_offset="0 0 0"
       mesh_name="ROS2_J2"
+      ixx="0.1338857818623325"
+      iyy="0.1338857818623325"
+      izz="0.0151074"
+      mass="8.393"
   />
   <xacro:create_link
@@ -26,4 +38,8 @@
       rpy_offset="0 0 0"
       mesh_name="ROS2_J3"
+      ixx="0.031209355099586295"
+      iyy="0.031209355099586295"
+      izz="0.004095"
+      mass="2.275"
   />
   <xacro:create_link
@@ -32,4 +48,8 @@
       rpy_offset="0 0 0"
       mesh_name="ROS2_J4"
+      ixx="0.0025598989760400002"
+      iyy="0.0025598989760400002"
+      izz="0.0021942"
+      mass="1.219"
   />
   <xacro:create_link
@@ -38,4 +58,8 @@
       rpy_offset="0 0 0"
       mesh_name="ROS2_J5"
+      ixx="0.0025598989760400002"
+      iyy="0.0025598989760400002"
+      izz="0.0021942"
+      mass="1.219"
   />
   <xacro:create_link
@@ -44,4 +68,8 @@
       rpy_offset="0 0 0"
       mesh_name="ROS2_J6"
+      ixx="9.890410052167731e-05"
+      iyy="9.890410052167731e-05"
+      izz="0.0001321171875"
+      mass="0.1879"
   />
   <link name="ft_frame"/>
@@ -58,5 +86,5 @@
     <origin xyz="0 0 0.117" rpy="0 0 0"/>
     <axis xyz="0 0 1"/>
-    <limit effort="1000.0" lower="${-pi}" upper="${pi}" velocity="2.5"/>
+    <limit effort="150.0" lower="-6.283185307179586" upper="6.283185307179586" velocity="3.141592653589793"/>
   </joint>
   <joint name="joint_2" type="revolute">
@@ -65,5 +93,5 @@
     <origin xyz="-0.081 0 0.101" rpy="0 ${-pi/2} 0"/>
     <axis xyz="0 0 1"/>
-    <limit effort="1000.0" lower="${-pi}" upper="${pi}" velocity="2.5"/>
+    <limit effort="150.0" lower="-6.283185307179586" upper="6.283185307179586" velocity="3.141592653589793"/>
   </joint>
   <joint name="joint_3" type="revolute">
@@ -72,5 +100,5 @@
     <origin xyz="0.35 0 -0.0035" rpy="${pi} 0 0"/>
     <axis xyz="0 0 1"/>
-    <limit effort="1000.0" lower="${-pi}" upper="${pi}" velocity="2.5"/>
+    <limit effort="80.0" lower="-3.141592653589793" upper="3.141592653589793" velocity="3.141592653589793"/>
   </joint>
   <joint name="joint_4" type="revolute">
@@ -79,5 +107,5 @@
     <origin xyz="0.0805 0 0.0775" rpy="0 ${pi/2} 0"/>
     <axis xyz="0 0 1"/>
-    <limit effort="1000.0" lower="${-pi}" upper="${pi}" velocity="2.5"/>
+    <limit effort="28.0" lower="-6.283185307179586" upper="6.283185307179586" velocity="3.141592653589793"/>
   </joint>
   <joint name="joint_5" type="revolute">
@@ -86,5 +114,5 @@
     <origin xyz="0 0 0.2695" rpy="0 ${-pi/2} 0"/>
     <axis xyz="0 0 1"/>
-    <limit effort="1000.0" lower="${-pi}" upper="${pi}" velocity="2.5"/>
+    <limit effort="28.0" lower="-6.283185307179586" upper="6.283185307179586" velocity="3.141592653589793"/>
   </joint>
   <joint name="joint_6" type="revolute">
@@ -93,5 +121,5 @@
     <origin xyz="0.1705 0 0" rpy="0 ${pi/2} 0"/>
     <axis xyz="0 0 1"/>
-    <limit effort="1000.0" lower="${-pi}" upper="${pi}" velocity="2.5"/>
+    <limit effort="28.0" lower="-6.283185307179586" upper="6.283185307179586" velocity="3.141592653589793"/>
   </joint>
   <joint name="joint-ft_frame" type="fixed">

Commit message: Fixed meshes not loading

File: urdf/inc/create_link.xacro (robot description, xacro)
@@ -14,5 +14,5 @@
         <origin xyz="${xyz_offset}" rpy="${rpy_offset}"/>
         <geometry>
-          <mesh filename="package://tr_robot_description/meshes/${mesh_name}.stl" scale="0.001 0.001 0.001"/>
+          <mesh filename="$(find tr_robot_description)/meshes/${mesh_name}.stl" scale="0.001 0.001 0.001"/>
         </geometry>
       </visual>
@@ -20,5 +20,5 @@
         <origin xyz="${xyz_offset}" rpy="${rpy_offset}"/>
         <geometry>
-          <mesh filename="package://tr_robot_description/meshes/${mesh_name}.stl" scale="0.001 0.001 0.001"/>
+          <mesh filename="$(find tr_robot_description)/meshes/${mesh_name}.stl" scale="0.001 0.001 0.001"/>
         </geometry>
       </collision>

Commit message: fixed mash loading

File: urdf/inc/create_link.xacro (robot description, xacro)
@@ -14,5 +14,5 @@
         <origin xyz="${xyz_offset}" rpy="${rpy_offset}"/>
         <geometry>
-          <mesh filename="$(find tr_robot_description)/meshes/${mesh_name}.stl" scale="0.001 0.001 0.001"/>
+          <mesh filename="file://$(find tr_robot_description)/meshes/${mesh_name}.stl" scale="0.001 0.001 0.001"/>
         </geometry>
       </visual>
@@ -20,5 +20,5 @@
         <origin xyz="${xyz_offset}" rpy="${rpy_offset}"/>
         <geometry>
-          <mesh filename="$(find tr_robot_description)/meshes/${mesh_name}.stl" scale="0.001 0.001 0.001"/>
+          <mesh filename="file://$(find tr_robot_description)/meshes/${mesh_name}.stl" scale="0.001 0.001 0.001"/>
         </geometry>
       </collision>
