Commit message: fixed typo

File: urdf/mercury_description.urdf.xacro (robot description, xacro)
@@ -81,5 +81,5 @@
     <axis xyz="0 0 1"/>
   </joint>
-  <joint name="joint_1" type="revolute">
+  <joint name="joint1" type="revolute">
     <parent link="base_link"/>
     <child link="link_1"/>
@@ -88,5 +88,5 @@
     <limit effort="150.0" lower="-6.283185307179586" upper="6.283185307179586" velocity="3.141592653589793"/>
   </joint>
-  <joint name="joint_2" type="revolute">
+  <joint name="joint2" type="revolute">
     <parent link="link_1"/>
     <child link="link_2"/>
@@ -95,5 +95,5 @@
     <limit effort="150.0" lower="-6.283185307179586" upper="6.283185307179586" velocity="3.141592653589793"/>
   </joint>
-  <joint name="joint_3" type="revolute">
+  <joint name="joint3" type="revolute">
     <parent link="link_2"/>
     <child link="link_3"/>
@@ -102,5 +102,5 @@
     <limit effort="80.0" lower="-3.141592653589793" upper="3.141592653589793" velocity="3.141592653589793"/>
   </joint>
-  <joint name="joint_4" type="revolute">
+  <joint name="joint4" type="revolute">
     <parent link="link_3"/>
     <child link="link_4"/>
@@ -109,5 +109,5 @@
     <limit effort="28.0" lower="-6.283185307179586" upper="6.283185307179586" velocity="3.141592653589793"/>
   </joint>
-  <joint name="joint_5" type="revolute">
+  <joint name="joint5" type="revolute">
     <parent link="link_4"/>
     <child link="link_5"/>
@@ -116,5 +116,5 @@
     <limit effort="28.0" lower="-6.283185307179586" upper="6.283185307179586" velocity="3.141592653589793"/>
   </joint>
-  <joint name="joint_6" type="revolute">
+  <joint name="joint6" type="revolute">
     <parent link="link_5"/>
     <child link="link_6"/>
